File: hard/Sound_Sheet.kicad_sch (KiCad schematic)
At the start: 39 parts, among them J3 Black headphone jack, U10 TLV9062, U11 MCP4251-xxxx-SL, U13 TLV9062, U14 TLV9062, U5 PCM5102A, U7 AP2112K-3.3

Commit message: Modifying paths
Parts:
- J3: footprint Connector_Audio:AUDIO-TH_320B -> easyeda2kicad:AUDIO-TH_320B
Changed lines of the file:
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@@
 			)
 		)
-		(property "Footprint" "Connector_Audio:AUDIO-TH_320B"
+		(property "Footprint" "easyeda2kicad:AUDIO-TH_320B"
 			(at 74.93 142.24 0)
 			(effects
