File: hard/Untitled.kicad_pcb (KiCad board)
At the start: 2 copper layers, 99.6 x 75.1 mm, 92 parts, among them IC2 MTCH6102-I_SS, J2 USB_C_Receptacle, J3 Black headphone jack, J5 TP1, J7 TP3, SW1 RotaryEncoder_Switch, SW90 BOOT, SW91 RESET, U1 RP2040, U10 TLV9062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

Commit message: Modifying paths
Parts:
- added R18: 27, Resistor_SMD:R_0402_1005Metric, F.Cu at (175.4, 90.3)
- J3: footprint Connector_Audio:AUDIO-TH_320B -> easyeda2kicad:AUDIO-TH_320B
Connections:
- U10 pad 4: GND -> (no net)
- U10 pad 8: +3V3A -> (no net)
- U13 pad 4: GND -> (no net)
- U13 pad 8: +3V3A -> (no net)
- U14 pad 4: GND -> (no net)
- U14 pad 8: +3V3A -> (no net)
